Commit message: enable grippers in robot model

File: yumiMatlab/yumi.urdf (robot description, URDF)
Before this commit: robot yumi, 20 links, 19 joints
Links:
- added link gripper_l_finger_l, mass 0.01; collision mesh filename=package://yumi_description/meshes/gripper/coarse/finger.stl; visual mesh filename=package://yumi_description/meshes/gripper/finger.stl
- added link gripper_r_finger_l, mass 0.01; collision mesh filename=package://yumi_description/meshes/gripper/coarse/finger.stl; visual mesh filename=package://yumi_description/meshes/gripper/finger.stl
Joints:
- added joint gripper_l_joint_m: type prismatic, parent gripper_l_base, child gripper_l_finger_l, origin xyz=0 0.0065 0.0837 rpy=0 0 0, axis 1 0 0, limit lower=0 upper=0.025 effort=20.0 velocity=0.02, mimic joint=gripper_l_joint
- added joint gripper_r_joint_m: type prismatic, parent gripper_r_base, child gripper_r_finger_l, origin xyz=0 0.0065 0.0837 rpy=0 0 0, axis 1 0 0, limit lower=0 upper=0.025 effort=20.0 velocity=0.02, mimic joint=gripper_r_joint
- joint gripper_l_joint: type fixed -> prismatic
- joint gripper_r_joint: limit lower=0 upper=0.025 effort=300 velocity=0.02 -> lower=0 upper=0.025 effort=20.0 velocity=0.02; type fixed -> prismatic
