Commit message: add custom sawyer message

File: yumiMatlab/sawyer.urdf (robot description, URDF)
Before this commit: robot sawyer, 33 links, 32 joints
Links:
- added link camera_base_link
- added link camera_bottom_screw_frame
- added link camera_link, mass 0.072; collision box size=0.02505 0.09 0.025; visual mesh filename=package://realsense2_description/meshes/d435.dae
- link head: geometry collision sphere radius=0.18; visual mesh filename=package://custom_sawyer_description/meshes/sawyer_pv/head.D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
- link pedestal: geometry collision cylinder length=0.62 radius=0.18; visual mesh filename=package://custom_sawyer_description/meshes/sawyer_pv/pedest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
- link right_arm_base_link: geometry collision cylinder length=0.24 radius=0.08; visual mesh filename=package://custom_sawyer_description/meshes/sawyer_pv/base.D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
- link right_l0: geometry collision sphere radius=0.07; visual mesh filename=package://custom_sawyer_description/meshes/sawyer_mp3/l0.DAE
- link right_l1: geometry collision sphere radius=0.07; visual mesh filename=package://custom_sawyer_description/meshes/sawyer_mp3/l1.DAE
- link right_l2: geometry collision cylinder length=0.34 radius=0.06; visual mesh filename=package://custom_sawyer_description/meshes/sawyer_pv/l2.DAE
- link right_l3: geometry collision sphere radius=0.06; visual mesh filename=package://custom_sawyer_description/meshes/sawyer_pv/l3.DAE
- link right_l4: geometry collision cylinder length=0.30 radius=0.045; visual mesh filename=package://custom_sawyer_description/meshes/sawyer_pv/l4.DAE
- link right_l5: geometry collision sphere radius=0.06; visual mesh filename=package://custom_sawyer_description/meshes/sawyer_pv/l5.DAE
- link right_l6: geometry collision cylinder length=0.05 radius=0.055; visual mesh filename=package://custom_sawyer_description/meshes/sawyer_mp1/l6.DAE
Joints:
- added joint camera_joint: type fixed, parent camera_base_link, child camera_bottom_screw_frame, origin xyz=0 0 0 rpy=0 0 0
- added joint camera_link_joint: type fixed, parent camera_bottom_screw_frame, child camera_link, origin xyz=0.010600000000000002 0.0175 0.0125 rpy=0 0 0
- added joint right_l6_to_camera: type fixed, parent right_l6, child camera_base_link, origin xyz=0 0.038279 0.028525 rpy=-1.57079632679 4.71238898 0, axis 0 0 0

Commit message: update robot mex

File: yumiMatlab/sawyer.urdf (robot description, URDF)
Before this commit: robot sawyer, 36 links, 35 joints
Links:
- link right_hand_camera: mass None -> 0.0
